Commit message: slightly modified

File: freight/freight_description/urdf/freight.gazebo.xacro (robot description, xacro)
@@ -1,10 +1,13 @@
 <?xml version="1.0"?>
 <robot name="turtlebot3_waffle" xmlns:xacro="http://ros.org/wiki/xacro">
-  <xacro:arg name="laser_visual"  default="true"/>
+  <!-- Parameters that allow us to see the rays from sensors -->
+  <xacro:arg name="laser_visual"  default="false"/>
   <xacro:arg name="camera_visual" default="false"/>
   <xacro:arg name="imu_visual"    default="false"/>
+  <!-- Base of the robot -->
   <gazebo reference="base_link">
     <material>Gazebo/DarkGrey</material>
   </gazebo>
+  <!-- Defining wheeel parameters -->
   <gazebo reference="wheel_left_link">
     <mu1>0.1</mu1>
@@ -27,22 +30,5 @@
     <material>Gazebo/FlatBlack</material>
   </gazebo>
-  <!-- <gazebo reference="caster_back_right_link">
-    <mu1>0.1</mu1>
-    <mu2>0.1</mu2>
-    <kp>1000000.0</kp>
-    <kd>100.0</kd>
-    <minDepth>0.001</minDepth>
-    <maxVel>1.0</maxVel>
-    <material>Gazebo/FlatBlack</material>
-  </gazebo>
-  <gazebo reference="caster_back_left_link">
-    <mu1>0.1</mu1>
-    <mu2>0.1</mu2>
-    <kp>1000000.0</kp>
-    <kd>100.0</kd>
-    <minDepth>0.001</minDepth>
-    <maxVel>1.0</maxVel>
-    <material>Gazebo/FlatBlack</material>
-  </gazebo> -->
+  <!-- Placing imu sensor where imu link is created  -->
   <gazebo reference="imu_link">
     <sensor type="imu" name="imu">
@@ -52,4 +38,5 @@
     <material>Gazebo/Grey</material>
   </gazebo>
+  <!-- Using the turtlebot differential drive controller to move fetch robot -->
   <gazebo>
     <plugin name="turtlebot3_waffle_controller" filename="libgazebo_ros_diff_drive.so">
@@ -74,4 +61,5 @@
     </plugin>
   </gazebo>
+  <!-- Defining the imu sensor parameters -->
   <gazebo>
     <plugin name="imu_plugin" filename="libgazebo_ros_imu.so">
@@ -102,4 +90,5 @@
     </plugin>
   </gazebo>
+  <!-- Defining 2d lidar parameters -->
   <gazebo reference="base_scan">
     <material>Gazebo/FlatBlack</material>
@@ -134,4 +123,5 @@
     </sensor>
   </gazebo>
+  <!-- Defining RGB-D camera parameters -->
   <gazebo reference="camera_rgb_frame">
     <sensor type="depth" name="realsense_R200">

File: freight/freight_description/urdf/freight.urdf.xacro (robot description, xacro)
@@ -7,10 +7,6 @@
   <xacro:property name="r200_cam_rgb_pz" value="0.013"/>
   <xacro:property name="r200_cam_depth_offset" value="0.01"/>
-  <!-- <link name="base_footprint"/>
-  <joint name="base_joint" type="fixed">
-    <parent link="base_footprint"/>
-    <child link="base_link" />
-    <origin xyz="0 0 0.005" rpy="0 0 0"/>
-  </joint> -->
+  <!-- All links and joints of robot are defined in this file -->
+  <!-- Base link of the robot -->
   <link name="base_link">
     <visual>
@@ -23,10 +19,5 @@
       </material>
     </visual>
-    <!-- <collision>
-      <origin rpy="0 0 0" xyz="0 0 0" />
-      <geometry>
-        <mesh filename="package://turtlebot3_description/meshes/freight/base_link_collision.STL" />
-      </geometry>
-    </collision> -->
+    <!-- Collision model of this link -->
     <collision>
       <origin xyz="0 0 0.175" rpy="0 0 0"/>
@@ -35,4 +26,5 @@
       </geometry>
     </collision>
+    <!-- inertial model of this link -->
     <inertial>
       <origin xyz="0 0 0.175" rpy="0 0 0"/>
@@ -43,4 +35,5 @@
     </inertial>
   </link>
+  <!-- Creating the joint between base and left wheel -->
   <joint name="wheel_left_joint" type="continuous">
     <parent link="base_link"/>
@@ -49,4 +42,5 @@
     <axis xyz="0 0 1"/>
   </joint>
+  <!-- Left wheel link -->
   <link name="wheel_left_link">
     <visual>
@@ -73,4 +67,5 @@
       </inertial>
   </link>
+  <!-- Right wheel joint -->
   <joint name="wheel_right_joint" type="continuous">
     <parent link="base_link"/>
@@ -79,4 +74,5 @@
     <axis xyz="0 0 1"/>
   </joint>
+  <!-- Right wheel link -->
   <link name="wheel_right_link">
     <visual>
@@ -103,44 +99,6 @@
       </inertial>
   </link>
-  <!-- <joint name="caster_back_right_joint" type="fixed">
-    <parent link="base_link"/>
-    <child link="caster_back_right_link"/>
-    <origin xyz="-0.177 -0.064 -0.004" rpy="-1.57 0 0"/>
-  </joint>
-  <link name="caster_back_right_link">
-    <collision>
-      <origin xyz="0 0.001 0" rpy="0 0 0"/>
-      <geometry>
-        <box size="0.030 0.009 0.020"/>
-      </geometry>
-    </collision>
-    <inertial>
-      <origin xyz="0 0 0" />
-      <mass value="0.005" />
-      <inertia ixx="0.001" ixy="0.0" ixz="0.0"
-               iyy="0.001" iyz="0.0"
-               izz="0.001" />
-    </inertial>
-  </link>
-  <joint name="caster_back_left_joint" type="fixed">
-    <parent link="base_link"/>
-    <child link="caster_back_left_link"/>
-    <origin xyz="-0.177 0.064 -0.004" rpy="-1.57 0 0"/>
-  </joint>
-  <link name="caster_back_left_link">
-    <collision>
-      <origin xyz="0 0.001 0" rpy="0 0 0"/>
-      <geometry>
-        <box size="0.030 0.009 0.020"/>
-      </geometry>
-    </collision>
-    <inertial>
-      <origin xyz="0 0 0" />
-      <mass value="0.005" />
-      <inertia ixx="0.001" ixy="0.0" ixz="0.0"
-               iyy="0.001" iyz="0.0"
-               izz="0.001" />
-    </inertial>
-  </link> -->
+  <!-- Defining links and joints for all snesors -->
+  <!-- IMU -->
   <joint name="imu_joint" type="fixed">
     <parent link="base_link"/>
@@ -149,4 +107,5 @@
   </joint>
   <link name="imu_link"/>
+  <!-- 2D LIDAR -->
   <joint name="scan_joint" type="fixed">
     <parent link="base_link"/>
@@ -176,4 +135,5 @@
     </inertial>
   </link>
+  <!-- RGBD Camera -->
   <joint name="camera_joint" type="fixed">
     <origin xyz="0.28 -0.064 0.138" rpy="0 0 0"/>
@@ -194,12 +154,4 @@
       </geometry>
     </collision>
-    <!-- This inertial field needs doesn't contain reliable data!! -->
-<!--   <inertial>
-      <mass value="0.564" />
-      <origin xyz="0 0 0" />
-      <inertia ixx="0.003881243" ixy="0.0" ixz="0.0"
-               iyy="0.000498940" iyz="0.0"
-               izz="0.003879257" />
-    </inertial>-->
   </link>
   <joint name="camera_rgb_joint" type="fixed">
